File: eagle/sensors.brd (EAGLE design)
At the start: 43 x 70 mm, 14 parts, among them U1 DHT22

Commit message: updates
Parts:
- added S1: (no value), switch-omron:B3F-10XX
- moved C1 10.5 mm to (35.6, 34.3)
Connections:
- net GND: now also S1.3
- net N$3: now also S1.1
Routing:
- net GND: track 148.6 -> 164.4 mm
- net VCC: track 104.9 -> 113.0 mm
- net N$3: track 10.2 -> 16.4 mm
- net N$12: track 26.5 -> 24.4 mm
- net N$10: track 13.9 -> 14.7 mm
Changed lines of the file:
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@@
 <param name="RoutingGrid" value="50mil"/>
 <param name="AutoGrid" value="1"/>
-<param name="Efforts" value="0"/>
+<param name="Efforts" value="2"/>
 <param name="TopRouterVariant" value="1"/>
 <param name="tpViaShape" value="round"/>
@@
 <element name="R1" library="SparkFun-Resistors" package="AXIAL-0.3EZ" value="10k" x="19.05" y="44.45" rot="R90"/>
 <element name="R2" library="SparkFun-Resistors" package="AXIAL-0.3EZ" value="10k" x="10.16" y="46.99" rot="R90"/>
-<element name="C1" library="SparkFun-Capacitors" package="CAP-PTH-5MM" value="100n" x="38.1" y="24.13" rot="R90"/>
+<element name="C1" library="SparkFun-Capacitors" package="CAP-PTH-5MM" value="100n" x="35.56" y="34.29" rot="R90"/>
 <element name="C2" library="SparkFun-Capacitors" package="CAP-PTH-5MM" value="100n" x="13.97" y="43.18" rot="R90"/>
 <element name="JP1" library="SparkFun-Connectors" package="1X06" value="FTDI" x="13.97" y="52.07" rot="R90"/>
@@
 <element name="C3" library="SparkFun-Capacitors" package="CAP-PTH-5MM" value="100n" x="21.59" y="53.34" rot="R180"/>
 <element name="U$1" library="dp_devices" package="DP7043_V1" value="" x="29.21" y="39.37" rot="R90"/>
+<element name="S1" library="switch-omron" package="B3F-10XX" value="" x="15.24" y="33.02">
+<attribute name="MF" value="" x="15.24" y="33.02" size="1.778" layer="27" display="off"/>
+<attribute name="OC_FARNELL" value="176432" x="15.24" y="33.02" size="1.778" layer="27" display="off"/>
+<attribute name="MPN" value="B3F-1000" x="15.24" y="33.02" size="1.778" layer="27" display="off"/>
+<attribute name="OC_NEWARK" value="36M3542" x="15.24" y="33.02" size="1.778" layer="27" display="off"/>
+</element>
 </elements>
 <signals>
@@
 <wire x1="16.51" y1="45.72" x2="16.51" y2="26.67" width="0.254" layer="1"/>
 <wire x1="19.05" y1="48.26" x2="16.51" y2="45.72" width="0.254" layer="1"/>
-<wire x1="38.1" y1="13.97" x2="38.1" y2="21.63" width="0.1524" layer="1"/>
 <wire x1="30.48" y1="25.4" x2="31.75" y2="24.13" width="0.1524" layer="16"/>
 <wire x1="15.24" y1="25.4" x2="20.32" y2="25.4" width="0.1524" layer="16"/>
 <wire x1="20.32" y1="25.4" x2="30.48" y2="25.4" width="0.1524" layer="16"/>
 <wire x1="13.97" y1="24.13" x2="15.24" y2="25.4" width="0.1524" layer="16"/>
-<wire x1="35.56" y1="19.05" x2="38.1" y2="21.59" width="0.1524" layer="16"/>
 <wire x1="26.67" y1="19.05" x2="35.56" y2="19.05" width="0.1524" layer="16"/>
 <wire x1="20.32" y1="25.4" x2="26.67" y2="19.05" width="0.1524" layer="16"/>
-<wire x1="38.1" y1="21.59" x2="38.1" y2="21.63" width="0.1524" layer="16"/>
 <wire x1="19.1209" y1="48.4277" x2="19.1209" y2="53.2526" width="0.1524" layer="16"/>
 <wire x1="19.1209" y1="53.2526" x2="19.09" y2="53.34" width="0.1524" layer="16"/>
@@
 <wire x1="34.1317" y1="65.9403" x2="34.29" y2="66.04" width="0.1524" layer="1"/>
 <wire x1="19.1209" y1="53.4313" x2="19.09" y2="53.34" width="0.1524" layer="1"/>
+<wire x1="35.5613" y1="28.7707" x2="35.5613" y2="31.6299" width="0.1524" layer="16"/>
+<wire x1="36.0974" y1="28.2346" x2="35.5613" y2="28.7707" width="0.1524" layer="16"/>
+<wire x1="36.0974" y1="19.657" x2="36.0974" y2="28.2346" width="0.1524" layer="16"/>
+<wire x1="35.5613" y1="19.1209" x2="36.0974" y2="19.657" width="0.1524" layer="16"/>
+<wire x1="35.5613" y1="31.6299" x2="35.56" y2="31.79" width="0.1524" layer="16"/>
+<wire x1="38.0631" y1="16.6191" x2="38.0631" y2="14.1173" width="0.1524" layer="16"/>
+<wire x1="35.5613" y1="19.1209" x2="38.0631" y2="16.6191" width="0.1524" layer="16"/>
+<wire x1="38.0631" y1="14.1173" x2="38.1" y2="13.97" width="0.1524" layer="16"/>
+<wire x1="35.5613" y1="19.1209" x2="35.56" y2="19.05" width="0.1524" layer="16"/>
 </signal>
 <signal name="N$2">
@@
 <wire x1="44.45" y1="15.24" x2="40.64" y2="11.43" width="0.254" layer="16"/>
 <wire x1="44.45" y1="15.24" x2="44.45" y2="15.6" width="0.254" layer="16"/>
-<wire x1="44.45" y1="17.78" x2="38.1" y2="26.63" width="0.254" layer="1"/>
-<wire x1="44.45" y1="15.6" x2="44.45" y2="17.78" width="0.254" layer="1"/>
 <wire x1="13.97" y1="64.77" x2="13.97" y2="62.23" width="0.254" layer="1"/>
 <wire x1="31.75" y1="48.26" x2="33.02" y2="48.26" width="0.254" layer="16"/>
@@
 <contactref element="R4" pad="2"/>
 <wire x1="38.1" y1="26.67" x2="38.1" y2="26.805" width="0.4064" layer="16"/>
-<wire x1="38.1" y1="26.805" x2="38.1" y2="43.18" width="0.4064" layer="16"/>
-<wire x1="38.1" y1="43.18" x2="33.7743" y2="48.26" width="0.4064" layer="16"/>
 <wire x1="33.7743" y1="48.26" x2="31.75" y2="48.26" width="0.4064" layer="16"/>
 <wire x1="33.7743" y1="48.26" x2="33.7743" y2="53.2526" width="0.1524" layer="16"/>
 <wire x1="33.7743" y1="53.2526" x2="33.75" y2="53.34" width="0.1524" layer="16"/>
 <wire x1="38.2418" y1="26.805" x2="38.1" y2="26.805" width="0.1524" layer="16"/>
-<wire x1="38.2418" y1="26.805" x2="38.1" y2="26.63" width="0.1524" layer="16"/>
+<contactref element="S1" pad="3"/>
+<wire x1="12.1516" y1="18.4061" x2="12.1516" y2="30.7364" width="0.1524" layer="1"/>
+<wire x1="13.9386" y1="16.6191" x2="12.1516" y2="18.4061" width="0.1524" layer="1"/>
+<wire x1="12.1516" y1="30.7364" x2="11.9888" y2="30.7594" width="0.1524" layer="1"/>
+<wire x1="13.9386" y1="16.6191" x2="13.97" y2="16.51" width="0.1524" layer="1"/>
+<wire x1="38.0631" y1="34.1317" x2="38.0631" y2="26.9837" width="0.1524" layer="16"/>
+<wire x1="35.5613" y1="36.6335" x2="38.0631" y2="34.1317" width="0.1524" layer="16"/>
+<wire x1="38.0631" y1="26.9837" x2="38.1" y2="26.805" width="0.1524" layer="16"/>
+<wire x1="35.5613" y1="36.6335" x2="35.56" y2="36.79" width="0.1524" layer="16"/>
+<wire x1="35.3826" y1="46.462" x2="35.3826" y2="36.8122" width="0.1524" layer="16"/>
+<wire x1="33.7743" y1="48.0703" x2="35.3826" y2="46.462" width="0.1524" layer="16"/>
+<wire x1="35.3826" y1="36.8122" x2="35.56" y2="36.79" width="0.1524" layer="16"/>
+<wire x1="33.7743" y1="48.0703" x2="33.7743" y2="48.26" width="0.1524" layer="16"/>
+<wire x1="38.2418" y1="21.8014" x2="38.2418" y2="26.6263" width="0.1524" layer="16"/>
+<wire x1="44.3176" y1="15.7256" x2="38.2418" y2="21.8014" width="0.1524" layer="16"/>
+<wire x1="38.2418" y1="26.6263" x2="38.1" y2="26.67" width="0.1524" layer="16"/>
+<wire x1="44.3176" y1="15.7256" x2="44.45" y2="15.6" width="0.1524" layer="16"/>
 </signal>
 <signal name="N$3">
@@
 <wire x1="19.05" y1="40.64" x2="13.97" y2="40.64" width="0.1524" layer="16"/>
 <wire x1="13.97" y1="40.64" x2="13.97" y2="40.68" width="0.1524" layer="16"/>
+<contactref element="S1" pad="1"/>
+<wire x1="12.1516" y1="38.7779" x2="12.1516" y2="35.3826" width="0.1524" layer="1"/>
+<wire x1="13.9386" y1="40.5649" x2="12.1516" y2="38.7779" width="0.1524" layer="1"/>
+<wire x1="12.1516" y1="35.3826" x2="11.9888" y2="35.2806" width="0.1524" layer="1"/>
+<wire x1="13.9386" y1="40.5649" x2="13.97" y2="40.68" width="0.1524" layer="1"/>
 </signal>
 <signal name="N$4">
@@
 <contactref element="NRF24L01+" pad="6"/>
 <contactref element="ATTINY84" pad="8"/>
-<wire x1="36.83" y1="27.94" x2="31.75" y2="33.02" width="0.254" layer="16"/>
-<wire x1="36.83" y1="22.86" x2="36.83" y2="27.94" width="0.254" layer="16"/>
-<wire x1="33.02" y1="22.86" x2="36.83" y2="22.86" width="0.254" layer="16"/>
+<wire x1="35.56" y1="27.94" x2="31.75" y2="33.02" width="0.254" layer="16"/>
+<wire x1="35.56" y1="22.86" x2="35.56" y2="27.94" width="0.254" layer="16"/>
+<wire x1="33.02" y1="22.86" x2="35.56" y2="22.86" width="0.254" layer="16"/>
 <wire x1="30.48" y1="20.32" x2="33.02" y2="22.86" width="0.254" layer="16"/>
 <wire x1="27.94" y1="20.32" x2="30.48" y2="20.32" width="0.254" layer="16"/>
@@
 <wire x1="27.94" y1="44.45" x2="27.94" y2="52.07" width="0.254" layer="16"/>
 <wire x1="27.94" y1="52.07" x2="29.21" y2="53.34" width="0.254" layer="16"/>
-<wire x1="29.21" y1="53.34" x2="29.75" y2="53.34" width="0" layer="19" extent="16-16"/>
+<wire x1="29.1281" y1="53.4313" x2="29.6642" y2="53.4313" width="0.1524" layer="16"/>
+<wire x1="29.6642" y1="53.4313" x2="29.75" y2="53.34" width="0.1524" layer="16"/>
+<wire x1="29.1281" y1="53.4313" x2="29.21" y2="53.34" width="0.1524" layer="16"/>
 </signal>
 <signal name="N$11">
