File: eagle/sensors.sch (EAGLE design)
At the start: 13 parts, among them U1 DHT22

Commit message: make capacitors bigger
Parts:
- C1, C2, C3: device SparkFun-Capacitors:CAPPTH -> SparkFun-Capacitors:CAPPTH1
Changed lines of the file:
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@@
 <part name="R1" library="SparkFun-Resistors" deviceset="RESISTOR" device="EZ" value="10k"/>
 <part name="R2" library="SparkFun-Resistors" deviceset="RESISTOR" device="EZ" value="10k"/>
-<part name="C1" library="SparkFun-Capacitors" deviceset="CAP" device="PTH" value="100n"/>
-<part name="C2" library="SparkFun-Capacitors" deviceset="CAP" device="PTH" value="100n"/>
+<part name="C1" library="SparkFun-Capacitors" deviceset="CAP" device="PTH1" value="100n"/>
+<part name="C2" library="SparkFun-Capacitors" deviceset="CAP" device="PTH1" value="100n"/>
 <part name="JP1" library="SparkFun-Connectors" deviceset="ARDUINO_SERIAL_PROGRAM" device="PTH" value="FTDI"/>
 <part name="GND2" library="supply1" deviceset="GND" device=""/>
@@
 <part name="P+1" library="supply1" deviceset="VCC" device=""/>
 <part name="U1" library="RHT03_DHT-22_AM2302" deviceset="RHT03_DHT-22_AM2302" device="" value="DHT22"/>
-<part name="C3" library="SparkFun-Capacitors" deviceset="CAP" device="PTH" value="100n"/>
+<part name="C3" library="SparkFun-Capacitors" deviceset="CAP" device="PTH1" value="100n"/>
 </parts>
 <sheets>

Commit message: board layout v1.1
Changed lines of the file:
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@@
 <?xml version="1.0" encoding="utf-8"?>
 <!DOCTYPE eagle SYSTEM "eagle.dtd">
-<eagle version="6.5.0">
+<eagle version="7.5.0">
 <drawing>
 <settings>
@@
 <setting verticaltext="up"/>
 </settings>
-<grid distance="0.1" unitdist="inch" unit="inch" style="dots" multiple="1" display="yes" altdistance="0.01" altunitdist="inch" altunit="inch"/>
+<grid distance="0.1" unitdist="inch" unit="inch" style="lines" multiple="1" display="no" altdistance="0.01" altunitdist="inch" altunit="inch"/>
 <layers>
 <layer number="1" name="Top" color="4" fill="1" visible="no" active="no"/>
@@
 <instance part="GND5" gate="1" x="76.2" y="33.02"/>
 <instance part="R4" gate="G$1" x="99.06" y="48.26" rot="R270"/>
-<instance part="GND6" gate="1" x="99.06" y="38.1"/>
+<instance part="GND6" gate="1" x="99.06" y="35.56"/>
 <instance part="P+1" gate="VCC" x="33.02" y="114.3"/>
 <instance part="U1" gate="G$1" x="58.42" y="43.18" rot="MR0"/>
@@
 <wire x1="73.66" y1="50.8" x2="73.66" y2="55.88" width="0.1524" layer="91"/>
 <junction x="73.66" y="50.8"/>
+<junction x="68.58" y="50.8"/>
 </segment>
 </net>
@@
 </segment>
 <segment>
-<pinref part="R4" gate="G$1" pin="P$2"/>
-<pinref part="GND6" gate="1" pin="GND"/>
-</segment>
-<segment>
 <pinref part="GND4" gate="1" pin="GND"/>
 <pinref part="NRF24L01+" gate="G$1" pin="1"/>
@@
 <wire x1="116.84" y1="73.66" x2="111.76" y2="73.66" width="0.1524" layer="91"/>
 <junction x="111.76" y="73.66"/>
+</segment>
+<segment>
+<pinref part="GND6" gate="1" pin="GND"/>
+<pinref part="R4" gate="G$1" pin="P$2"/>
+<wire x1="99.06" y1="38.1" x2="99.06" y2="40.64" width="0.1524" layer="91"/>
 </segment>
 </net>
@@
 <wire x1="127" y1="63.5" x2="132.08" y2="63.5" width="0.1524" layer="91"/>
 <wire x1="132.08" y1="63.5" x2="132.08" y2="86.36" width="0.1524" layer="91"/>
-</segment>
-</net>
-<net name="N$10" class="0">
-<segment>
-<pinref part="R4" gate="G$1" pin="P$1"/>
-<wire x1="99.06" y1="55.88" x2="99.06" y2="71.12" width="0.1524" layer="91"/>
-<pinref part="ATTINY84" gate="G$1" pin="(PCINT1/AIN0/ADC1)PA1"/>
-<wire x1="99.06" y1="71.12" x2="93.98" y2="71.12" width="0.1524" layer="91"/>
 </segment>
 </net>
@@
 </segment>
 </net>
+<net name="N$10" class="0">
+<segment>
+<pinref part="ATTINY84" gate="G$1" pin="(PCINT1/AIN0/ADC1)PA1"/>
+<wire x1="93.98" y1="71.12" x2="99.06" y2="71.12" width="0.1524" layer="91"/>
+<pinref part="R4" gate="G$1" pin="P$1"/>
+<wire x1="99.06" y1="71.12" x2="99.06" y2="55.88" width="0.1524" layer="91"/>
+</segment>
+</net>
 </nets>
 </sheet>
 </sheets>
+<errors>
+</errors>
 </schematic>
 </drawing>

Commit message: updates
Parts:
- added S1: (no value), switch-omron:10-XX
Connections:
- net GND: now also S1.P
- net N$3: now also S1.S
Changed lines of the file:
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@@
 <part name="U1" library="RHT03_DHT-22_AM2302" deviceset="RHT03_DHT-22_AM2302" device="" value="DHT22"/>
 <part name="C3" library="SparkFun-Capacitors" deviceset="CAP" device="PTH1" value="100n"/>
+<part name="S1" library="switch-omron" deviceset="10-XX" device=""/>
 </parts>
 <sheets>
@@
 <instance part="U1" gate="G$1" x="58.42" y="43.18" rot="MR0"/>
 <instance part="C3" gate="G$1" x="121.92" y="73.66" rot="R90"/>
+<instance part="S1" gate="1" x="124.46" y="109.22" rot="R90"/>
 </instances>
 <busses>
@@
 <junction x="134.62" y="86.36"/>
 <junction x="134.62" y="83.82"/>
+<pinref part="S1" gate="1" pin="P"/>
+<wire x1="129.54" y1="109.22" x2="132.08" y2="109.22" width="0.1524" layer="91"/>
+<wire x1="132.08" y1="109.22" x2="132.08" y2="88.9" width="0.1524" layer="91"/>
+<wire x1="132.08" y1="88.9" x2="134.62" y2="88.9" width="0.1524" layer="91"/>
+<junction x="134.62" y="88.9"/>
 </segment>
 <segment>
@@
 <wire x1="93.98" y1="99.06" x2="96.52" y2="99.06" width="0.1524" layer="91"/>
 <pinref part="R1" gate="G$1" pin="1"/>
-<wire x1="96.52" y1="99.06" x2="109.22" y2="99.06" width="0.1524" layer="91"/>
+<wire x1="96.52" y1="99.06" x2="104.14" y2="99.06" width="0.1524" layer="91"/>
 <junction x="96.52" y="99.06"/>
+<wire x1="104.14" y1="99.06" x2="109.22" y2="99.06" width="0.1524" layer="91"/>
+<wire x1="104.14" y1="99.06" x2="104.14" y2="109.22" width="0.1524" layer="91"/>
+<pinref part="S1" gate="1" pin="S"/>
+<wire x1="104.14" y1="109.22" x2="119.38" y2="109.22" width="0.1524" layer="91"/>
+<junction x="104.14" y="99.06"/>
 </segment>
 </net>
